File: avr-breadboard.kicad_pcb (KiCad board)
At the start: 2 copper layers, 33.1 x 42.9 mm, 10 parts, among them J1 Conn_01x08, J2 Conn_01x02, J3 Conn_02x03_Counter_Clockwise, SW1 SW_Push, U1 ATtiny13-20PU, Y1 Crystal

Commit message: Update
Parts:
- J1: footprint Connector_PinHeader_2.00mm:PinHeader_1x08_P2.00mm_Vertical -> Connector_PinSocket_2.54mm:PinSocket_1x08_P2.54mm_Vertical
- J2: footprint Connector_PinSocket_2.00mm:PinSocket_1x02_P2.00mm_Vertical -> Connector_PinSocket_2.54mm:PinSocket_1x02_P2.54mm_Vertical
- J3: footprint Connector_PinSocket_2.00mm:PinSocket_2x03_P2.00mm_Vertical -> Connector_PinSocket_2.54mm:PinSocket_2x03_P2.54mm_Vertical
- moved J3 1.07 mm to (132.3, 73.7)
- moved J2 0.85 mm to (129.2, 94.9)
Routing:
- net GND: track 13.0 -> 80.0 mm, vias 1 -> 9
- net MOSI: track 75.9 -> 77.8 mm
- net PB3: track 50.0 -> 51.7 mm
- net PB4: track 51.1 -> 51.9 mm
- net MISO: track 76.2 -> 76.7 mm
- net RESET: track 45.9 -> 45.8 mm, vias 0 -> 2
Other:
- board size 33.1 x 42.9 mm -> 33.2 x 47.9 mm
- board text added: "Alejandro Gallo 2020"
- board text added: "PCINT0|AIN0 MOSI PB0"
- board text added: "PCINT1|INT0|AIN1 MISO PB1"
- board text added: "PCINT2|T0|ADC1 SCK PB2"
- board text added: "PCINT5|ADC0 RST PB5"
- board text removed: "PCINT0|AIN0 PB0"
- board text removed: "PCINT1|INT0|AIN1 PB1"
- board text removed: "PCINT2|T0|ADC1 PB2"
- board text removed: "PCINT5|ADC0 PB5"
